File: Hardware/monitoring_system_schematic/monitoring_system_schematic.kicad_sch (KiCad schematic)
At the start: 7 parts, among them U2 DS18B20, U4 DS18B20

Commit message: Rev A routed and complete for the schematic
Parts:
- removed U1: ~, symbol custom_symbols:Raspberry_Pi_Zero
- removed U2, U4: DS18B20, Package_TO_SOT_THT:TO-92_Inline, symbol Sensor_Temperature:DS18B20
- removed U3: ~, symbol custom_symbols:Bus_Bar
- removed U5: ~, symbol custom_symbols:TTL_to_RS232
- removed U6: ~, symbol custom_symbols:battery_bank
- removed U7: ~, symbol custom_symbols:USB_bulkhead
- added C1, C2, C3, C4, C5, C6, C7, C8, C9: 0.1u, lcsc_footprints:C307331_C0402, symbol Device:C_Small
- added H1, H2, H3, H4: MountingHole, MountingHole:MountingHole_2.7mm_M2.5_Pad_Via, symbol Mechanical:MountingHole
- added J1: RaspberryPi_GPIO_40W, footprints:RPi_Zero_ModelB_40W_Carrier, symbol RaspberryPi:RaspberryPi_GPIO_40W
- added J2, J3: Conn_01x02, Connector_PinHeader_2.54mm:PinHeader_1x02_P2.54mm_Vertical, symbol Connector_Generic:Conn_01x02
- added JP1, JP2, JP3, JP4: SldJmp, Jumper:SolderJumper-2_P1.3mm_Open_RoundedPad1.0x1.5mm, symbol Jumper:SolderJumper_2_Open
- added R1, R2, R7, R8: 4.7k, lcsc_footprints:C25900_R0402, symbol Device:R_Small_US
- added R3, R4, R5, R6: 165, lcsc_footprints:C706217_R0805, symbol Device:R_Small_US
- added RJ1: PCB-6P6C-90_C189747, lcsc_footprints:C189747_RJ11-TH_PCB-6P6C-90, symbol lcsc_imported:PCB-6P6C-90_C189747
- added U1: ADS1115, lcsc_footprints:C37593_MSOP-10_L3_0-W3_0-P0_50-LS5_0-BL, symbol lcsc_imported:16-Bit_ADC_with_Integrated_Multiplexer,_PGA,_Comparator,_Oscillat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
- added U2: MAX3232CDR-JSM, lcsc_footprints:C46596312_SOIC-16_L9_9-W3_9-P1_27-LS6_1-BL, symbol lcsc_imported:MAX3232CDR-JSM
- added U3, U4, U5, U6: 5501-88011111, lcsc_footprints:C3097726_RJ45-TH_FRJ45017-1100G1K0200, symbol lcsc_imported:5501-88011111
- added U7: XL-0807RGBC-WS2812B, lcsc_footprints:C3646929_LED-SMD_4P-L2_0-W1_8_XL-0807RGBC-WS2812B, symbol lcsc_imported:XL-0807RGBC-WS2812B
Connections:
- net FREEZER_TEMP: now also J1.29 (GPIO5), R2.1, U3.7
- net FRIDGE_TEMP: now also J1.31 (GPIO6), R1.2, U3.3
- net GND: now also C1.1, C3.1, C5.1, C6.1, C7.1, C8.1, C9.1, J1.14 (GND), J1.20 (GND), J1.25 (GND), J1.30 (GND), J1.34 (GND), J1.39 (GND), J1.6 (GND), J1.9 (GND), R3.2, R4.2, R5.2, R6.2, RJ1.3, U1.1 (ADDR), U1.3 (GND), U2.15 (GND), U3.2, U3.6, U4.2, U4.6, U5.2, U5.6, U6.2, U6.6, U7.2 (GND)
- net RX: now also J1.10 (GPIO15/RXD0), J3.2 (Pin_2), U2.12 (ROUT1)
- net TX: now also J1.8 (GPIO14/TXD0), J3.1 (Pin_1), U2.11 (DIN1)
- new net: JP3.1 (A), R5.1
- new net: J1.12 (GPIO18/PWM0), U7.3 (DIN)
- new net: JP1.1 (A), R3.1
- new net: C5.2, U2.6 (V-)
- new net: JP2.1 (A), R4.1
- new net: JP4.1 (A), R6.1
- new net: C2.1, U2.3 (C1-)
- new net: C2.2, U2.1 (C1+)
- new net: J2.2 (Pin_2), RJ1.1, U2.13 (RIN1)
- new net: J2.1 (Pin_1), RJ1.2, U2.14 (DOUT1)
- new net: C3.2, U2.2 (V+)
- new net: C4.2, U2.4 (C2+)
- new net: C4.1, U2.5 (C2-)
- new net 3V3: C1.2, C6.2, C7.2, C8.2, J1.1 (3V3), J1.17 (3V3), R1.1, R2.2, R7.1, R8.1, U1.8 (VDD), U2.16 (VCC), U3.1, U3.5, U5.1, U5.5, U6.1, U6.5
- new net 5V: C9.2, J1.2 (5V), J1.4 (5V), U7.4 (VDD)
- new net ADC_ALERT: J1.7 (GPIO4/GPCLK0), U1.2 (ALERT/RDY)
- new net AIN0: JP1.2 (B), U1.4 (AIN0), U5.7
- new net AIN1: JP2.2 (B), U1.5 (AIN1), U5.8
- new net AIN2: JP3.2 (B), U1.6 (AIN2), U5.4
- new net AIN3: JP4.2 (B), U1.7 (AIN3), U5.3
- new net FREEZER_NC: J1.38 (GPIO20/MOSI1), U4.8
- new net FREEZER_NO: J1.36 (GPIO16), U4.7
- new net FRIDGE_NC: J1.35 (GPIO19/MISO1), U4.4
- new net FRIDGE_NO: J1.37 (GPIO26), U4.3
- new net GPIO0: J1.11 (GPIO17), U6.3
- new net GPIO1: J1.13 (GPIO27), U6.4
- new net GPIO2: J1.15 (GPIO22), U6.7
- new net GPIO3: J1.16 (GPIO23), U6.8
- new net SCL: J1.5 (GPIO3/SCL1), R7.2, U1.10 (SCL)
- new net SDA: J1.3 (GPIO2/SDA1), R8.2, U1.9 (SDA)
- no-connect marks 0 -> 5
Other:
- company: (none) -> LA Solarpunk
- title: (none) -> Solar Fridge Montitor Schematic
